File: PPQCU_CAD/Quadcopter.kicad_pcb (KiCad board)
At the start: 2 copper layers, 135.6 x 80.8 mm, 155 parts, among them P1 Battery, P10 CONN_02X04, P2 DEBUG, P3 Serv1, P4 Serv2, P5 Serv3, P6 Serv4, P7 SecServ1, P8 SecServ2, P9 ws2812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

Commit message: 4 layer version of board. Not used. Only kept for historical purposes
Parts:
- added TF3: GND, Measurement_Points:Measurement_Point_Round-SMD-Pad_Small, F.Cu at (84.2, 109.3)
- moved TF7 52.1 mm to (137.6, 81.0)
- moved TF4 50.5 mm to (137.0, 89.9)
- moved C12 49.1 mm to (86.1, 80.5)
- moved C2 49.1 mm to (135.1, 48.3)
- moved C22 49.1 mm to (138.9, 98.0)
- moved C26 49.1 mm to (129.5, 81.8)
- moved C28 49.1 mm to (86.1, 94.9)
- moved P1 49.1 mm to (101.6, 43.2)
- moved P9 49.1 mm to (83.8, 118.1)
- moved R1 49.1 mm to (140.5, 48.5)
- moved R11 49.1 mm to (116.7, 48.3)
- moved R12 49.1 mm to (116.7, 53.3)
- moved TF1 49.1 mm to (144.3, 61.5)
- moved TF31 49.1 mm to (128.8, 91.9)
- moved TF32 49.1 mm to (130.2, 109.1)
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Routing:
- net +3V3: track 383.5 -> 192.4 mm, vias 20 -> 12
- net GND: track 303.6 -> 379.6 mm, vias 33 -> 17
- net i2cDAT: track 177.7 -> 182.9 mm, vias 6 -> 7
- net Net-(R1-Pad1): track 12.4 -> 16.1 mm
- net WS_sig: track 131.4 -> 133.9 mm
- net aMISO: track 30.6 -> 28.3 mm
- net Net-(P7-Pad3): track 20.2 -> 19.4 mm
- net wIRQ: track 43.8 -> 44.6 mm
- net Net-(P8-Pad3): track 35.6 -> 34.9 mm
- net ServIntRD: track 82.5 -> 83.3 mm
- added copper zone on In2.Cu, net +3V3
- added copper zone on In1.Cu, net GND
- removed copper zone on F.Cu, net +3V3
- removed copper zone on B.Cu, net GND
Other:
- copper layers 2 -> 4
- net class Default: clearance 0.2 -> 0.05
- net class Power: clearance 0.2 -> 0.05
- rule pad_to_mask_clearance: 0.02 -> 0.05
- rule trace_clearance: 0.2 -> 0.05
- rule trace_min: 0.152 -> 0.25
- rule via_min_drill: 0.38 -> 0.3
- board text removed: "1 - SIG 2 - 5V 3 - GND"
- board text removed: "1 2 3"
- board text removed: "5V"
- board text removed: "GND"
- board text removed: "Motor BL"
- board text removed: "Motor BR"
- board text removed: "Motor FL"
- board text removed: "Motor FR"
- board text removed: "Philipp Schilk Quadcopter Controler Production 1 PP 2015/16"
- board text removed: "RGB Pinout:"
- board text removed: "SIG"
- board text removed: "Servo Pinout:"
- board text removed: "Thanks Mr. Esmail!"
